File: RotarySystem.sch (KiCad schematic (older format))
At the start: 7 parts

Commit message: Created the relay control board for the automated system.
Parts:
- gave numbers to parts that had none: 5
- renumbered PWR+ to PWR+1, PWR- to PWR-1
Connections:
- no-connect marks 0 -> 3
Changed lines of the file:
@@
-EESchema Schematic File Version 2  date Thu 07 Aug 2014 06:50:15 PM EDT
+EESchema Schematic File Version 2  date Fri 08 Aug 2014 01:11:47 AM EDT
 LIBS:power
 LIBS:device
@@
 Sheet 1 1
 Title "noname.sch"
-Date "7 aug 2014"
+Date "8 aug 2014"
 Rev ""
 Comp ""
@@
 Comment4 ""
 $EndDescr
+NoConn ~ 3750 4800
+NoConn ~ 1450 3450
+NoConn ~ 1450 3450
 Wire Wire Line
 	1950 4300 1950 3600
@@
 	1950 3600 1700 3600
 $Comp
-L CONN_1 PWR-
+L CONN_1 PWR-1
 U 1 1 53E4021D
 P 2450 5100
-F 0 "PWR-" H 2530 5100 40  0000 L CNN
+F 0 "PWR-1" H 2530 5100 40  0000 L CNN
 F 1 "CONN_1" H 2450 5155 30  0001 C CNN
 	1    2450 5100
@@
 $EndComp
 $Comp
-L CONN_1 PWR+
+L CONN_1 PWR+1
 U 1 1 53E40215
 P 2400 3050
-F 0 "PWR+" H 2480 3050 40  0000 L CNN
+F 0 "PWR+1" H 2480 3050 40  0000 L CNN
 F 1 "CONN_1" H 2400 3105 30  0001 C CNN
 	1    2400 3050
@@
 $EndComp
 $Comp
-L POT RV?
+L POT RV1
 U 1 1 53E3FFFA
 P 1700 3450
-F 0 "RV?" H 1700 3350 50  0000 C CNN
+F 0 "RV1" H 1700 3350 50  0000 C CNN
 F 1 "POT" H 1700 3450 50  0000 C CNN
 	1    1700 3450
@@
 $EndComp
 $Comp
-L R R?
+L R R3
 U 1 1 53E3FFF0
 P 2900 4550
-F 0 "R?" V 2980 4550 50  0000 C CNN
+F 0 "R3" V 2980 4550 50  0000 C CNN
 F 1 "R" V 2900 4550 50  0000 C CNN
 	1    2900 4550
@@
 $EndComp
 $Comp
-L R R?
+L R R1
 U 1 1 53E3FFEC
 P 1950 4550
-F 0 "R?" V 2030 4550 50  0000 C CNN
+F 0 "R1" V 2030 4550 50  0000 C CNN
 F 1 "R" V 1950 4550 50  0000 C CNN
 	1    1950 4550
@@
 $EndComp
 $Comp
-L R R?
+L R R2
 U 1 1 53E3FFE6
 P 2900 3700
-F 0 "R?" V 2980 3700 50  0000 C CNN
+F 0 "R2" V 2980 3700 50  0000 C CNN
 F 1 "R" V 2900 3700 50  0000 C CNN
 	1    2900 3700
@@
 $EndComp
 $Comp
-L BNC P?
+L BNC P1
 U 1 1 53E3EEE2
 P 2450 3750
-F 0 "P?" H 2460 3870 60  0000 C CNN
+F 0 "P1" H 2460 3870 60  0000 C CNN
 F 1 "BNC" V 2560 3690 40  0000 C CNN
 	1    2450 3750
