File: RelayControl.sch (KiCad schematic (older format))
At the start: 7 parts

Commit message: Reverted TS Electrical System.brd back to its original form from commit 0990b8f0af16a02e1b40e643ada236dd4e43b09a and also created extra brd files for the relaycontrol board and rotary system.
Parts:
- gave numbers to parts that had none: 1
Changed lines of the file:
@@
-EESchema Schematic File Version 2  date Fri 08 Aug 2014 01:41:24 AM EDT
+EESchema Schematic File Version 2  date Fri 08 Aug 2014 01:48:35 AM EDT
 LIBS:power
 LIBS:device
@@
 $EndDescr
 $Comp
-L NPN Q?
+L NPN Q1
 U 1 1 53E462E6
 P 4150 3000
-F 0 "Q?" H 4150 2850 50  0000 R CNN
+F 0 "Q1" H 4150 2850 50  0000 R CNN
 F 1 "NPN" H 4150 3150 50  0000 R CNN
 	1    4150 3000
